Commit message: feat : additional arm urdf + UR5 model

File: src/lex_simulation/robot_description/control/diff_drive.xacro (robot description, xacro)
@@ -2,5 +2,5 @@
 <robot name="diff_drive_controller" xmlns:xacro="http://www.ros.org/wiki/xacro">
     <!-- Differential drive controller macro -->
-    <xacro:macro name="diff_drive_controller">
+    <xacro:macro name="diff_drive_controller" params="wheel_separation wheel_diameter">
         <!-- Gazebo differential drive plugin -->
         <gazebo>
@@ -10,6 +10,6 @@
                 <rightJoint>right_wheel_joint</rightJoint>
                 <!-- Wheel properties -->
-                <wheelSeparation>0.5</wheelSeparation>
-                <wheelDiameter>0.12</wheelDiameter>
+                <wheelSeparation>${wheel_separation}</wheelSeparation>
+                <wheelDiameter>${wheel_diameter}</wheelDiameter>
                 <!-- Topic names -->
                 <commandTopic>cmd_vel</commandTopic>
@@ -29,5 +29,5 @@
                 <!-- Publish odometry TF -->
                 <publishOdomTF>true</publishOdomTF>
-                <publishWheelTF>false</publishWheelTF>
+                <publishWheelTF>true</publishWheelTF>
                 <!-- Odometry noise -->
                 <odometry_covariance_x>0.0001</odometry_covariance_x>

File: src/lex_simulation/robot_description/lex_robot_description.urdf.xacro (robot description, xacro)
@@ -71,4 +71,4 @@
         <mu2 value="0.5" />
     </gazebo>
-    <xacro:diff_drive_controller />
+    <xacro:diff_drive_controller wheel_separation="${2 * (body_radius + wheel_width/2)}" wheel_diameter="${2 * wheel_radius}" />
 </robot>

File: src/lex_simulation/robot_description/sensors/lidar.xacro (robot description, xacro)
@@ -36,5 +36,5 @@
             <sensor type="ray" name="lidar_sensor">
                 <pose>0 0 0 0 0 0</pose>
-                <visualize>true</visualize>
+                <visualize>false</visualize>
                 <update_rate>10</update_rate>
                 <ray>
