Commit message: feat : new map (warehouse), costmap redefinition

File: src/lex_simulation/urdf/lex_base/common/wheel.xacro (robot description, xacro)
@@ -62,6 +62,6 @@
         </transmission>
         <gazebo reference="${prefix}_wheel">
-            <mu1>15.0</mu1>
-            <mu2>15.0</mu2>
+            <mu1>50.0</mu1>
+            <mu2>50.0</mu2>
             <kp>1000000.0</kp>
             <kd>100.0</kd>

File: src/lex_simulation/urdf/lex_base/control/diff_drive.xacro (robot description, xacro)
@@ -25,5 +25,5 @@
                 <commandTimeout>0.5</commandTimeout>
                 <!-- Wheel torque limits -->
-                <maxWheelTorque>10</maxWheelTorque>
+                <maxWheelTorque>100</maxWheelTorque>
                 <maxWheelAcceleration>1.0</maxWheelAcceleration>
                 <!-- Publish odometry TF -->

File: src/lex_simulation/urdf/lex_robot_with_ur3e.urdf.xacro (robot description, xacro)
@@ -4,5 +4,5 @@
     <xacro:include filename="$(find lex_simulation)/urdf/ur3e/gazebo/gazebo_ur_macro.xacro" />
     <!-- UR3e arm parameters -->
-    <xacro:property name="arm_mount_offset_z" value="0.25" />
+    <xacro:property name="arm_mount_offset_z" value="0.15" />
     <xacro:property name="arm_mount_offset_x" value="0.0" />
     <xacro:property name="arm_mount_offset_y" value="0.0" />
